Commit message: edited inv doors

File: assets/urdf/door_test/door_2_inv_wall_2.urdf (robot description, URDF)
Before this commit: robot door_test, 5 links, 4 joints
Joints:
- joint base_joint: origin xyz=0 0.5 0.0 rpy=0 0 3.14159 -> xyz=0 -0.5 0.0 rpy=0 0 0
- joint door_handle: axis 1 0 0 -> -1 0 0; origin xyz=0.035 0.75 -1.02 -> xyz=0.035 0.75 -1.0
- joint door_hinge: limit lower=0 upper=1.57 effort=10000 velocity=100.00 -> lower=0 upper=1.57 effort=100 velocity=100.00; origin xyz=-0.07 0.06858 2.040 -> xyz=0.025 0.06858 0 rpy=0 3.14159 0
