Commit message: add new doors

File: assets/urdf/door_test/v2_door_left_1.urdf (robot description, URDF)
Before this commit: robot door_test, 5 links, 4 joints
Links:
- link door_handles: geometry collision mesh filename=./meshes/DH-02201_collision.dae scale=1.0 1.0 1.0; collision mesh filename=./meshes/DH-02201_collision.dae scale=1.0 1.0 1.0
- link door_latch: geometry collision box size=0.001 0.14 0.01
Joints:
- joint base_joint: origin xyz=0 -0.5 0.0 rpy=0 0 0 -> xyz=0 0.5 0.0 rpy=0 0 3.14159
- joint door_handle: axis -1 0 0 -> 1 0 0; origin xyz=0.035 0.75 -1.02 -> xyz=0.035 0.6 -1.35
- joint door_hinge: origin xyz=-0.07 0.972 0 rpy=3.14159 0 0 -> xyz=-0.07 0.06858 2.040

File: assets/urdf/door_test/v3_door_left_1.urdf (robot description, URDF)
Before this commit: robot door_test, 5 links, 4 joints
Links:
- removed link door_frame
- added link door_wall, mass 10000.0; collision box size=0.05029 0.06858 2.10820; collision box size=0.08 1.5 2.04
- link door_handles: geometry collision mesh filename=./meshes/with_plate_collision.dae scale=0.04 0.04 0.04; visual mesh filename=./meshes/with_plate.dae scale=0.04 0.04 0.04
Joints:
- joint base_joint: child door_frame -> door_wall; origin xyz=0 -0.5 0.0 rpy=0 0 0 -> xyz=0 0.5 0.0 rpy=0 0 3.14159
- joint door_handle: axis -1 0 0 -> 1 0 0; origin xyz=0.035 0.75 -1.0 -> xyz=0.035 0.75 -1.02
- joint door_hinge: limit lower=0 upper=1.57 effort=100 velocity=100.00 -> lower=0 upper=1.57 effort=10000 velocity=100.00; origin xyz=0.025 0.06858 0 rpy=0 3.14159 0 -> xyz=-0.07 0.06858 2.040; parent door_frame -> door_wall

File: assets/urdf/door_test/v4_door_left_1.urdf (robot description, URDF)
Before this commit: robot door_test, 5 links, 4 joints
Links:
- removed link door_frame
- added link door_wall, mass 10000.0; collision box size=0.05029 0.06858 2.10820; collision box size=0.08 1.5 2.04
- link door_handles: geometry collision mesh filename=./meshes/handle_5_collision.dae scale=0.04 0.04 0.04; visual mesh filename=./meshes/handle_5.dae scale=0.04 0.04 0.04
Joints:
- joint base_joint: child door_frame -> door_wall; origin xyz=0 -0.5 0.0 rpy=0 0 0 -> xyz=0 0.5 0.0 rpy=0 0 3.14159
- joint door_hinge: parent door_frame -> door_wall

Commit message: edit v3_door

File: assets/urdf/door_test/v2_door_left_1.urdf (robot description, URDF)
Before this commit: robot door_test, 5 links, 4 joints
Links:
- link door_handles: geometry collision mesh filename=./meshes/DH-02201_collision.dae scale=1.25 1.25 1.25; visual mesh filename=./meshes/DH-02201.dae scale=1.25 1.25 1.25
Joints:
- joint door_handle: origin xyz=0.035 0.6 -1.35 -> xyz=0.035 0.7 -1.25

File: assets/urdf/door_test/v3_door_left_1.urdf (robot description, URDF)
Before this commit: robot door_test, 5 links, 4 joints
Links:
- link door: geometry collision mesh filename=./meshes/door.dae; collision mesh filename=./meshes/plate_collision.dae scale=0.04 0.04 0.04
- link door_handles: geometry collision mesh filename=./meshes/handle_with_plate_collision.dae scale=0.04 0.04 0.04; visual mesh filename=./meshes/handle_with_plate.dae scale=0.04 0.04 0.04

Commit message: add other handles

File: assets/urdf/door_test/v2_door_left_1.urdf (robot description, URDF)
Before this commit: robot door_test, 5 links, 4 joints
Links:
- link door_handles: geometry collision mesh filename=./meshes/DH.stl scale=1.25 1.25 1.25; visual mesh filename=./meshes/DH-02201.dae scale=1.25 1.25 1.25

File: assets/urdf/door_test/v3_door_left_1.urdf (robot description, URDF)
Before this commit: robot door_test, 5 links, 4 joints
Links:
- link door: geometry collision mesh filename=./meshes/door.dae; collision mesh filename=./meshes/plate_collision.dae scale=0.035 0.035 0.035
- link door_handles: geometry collision mesh filename=./meshes/handle_with_plate.stl scale=0.035 0.035 0.035; visual mesh filename=./meshes/handle_with_plate.dae scale=0.035 0.035 0.035

File: assets/urdf/door_test/v4_door_left_1.urdf (robot description, URDF)
Before this commit: robot door_test, 5 links, 4 joints
Links:
- link door: geometry collision mesh filename=./meshes/door.dae; visual mesh filename=./meshes/door.dae
- link door_handles: geometry collision mesh filename=./meshes/v5.stl scale=0.04 0.04 0.04; visual mesh filename=./meshes/v5_handle.dae scale=0.04 0.04 0.04
